File: OpenFlops.kicad_sch (KiCad schematic)
At the start: 48 parts, among them J1 Conn_02x25_Odd_Even, J2 SWD, J3 BOOT 1/0, P1 ST-TF-003A, Q1 BSS138, SW1 RESET, U1 LM1117-3.3, U2 AT32F435RGT7, U3 74LS07, U4 OLED-0.91-128x32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

Commit message: Update to v1.1
Parts:
- added BZ1: Buzzer, Buzzer_Beeper:MagneticBuzzer_PUI_AT-0927-TT-6-R, symbol Device:Buzzer
- added D1: LL4148, Diode_SMD:D_MiniMELF, symbol Diode:LL4148
- added Q2: MMBT3904, Package_TO_SOT_SMD:SOT-23, symbol Transistor_BJT:MMBT3904
- added R22: 1K, Resistor_SMD:R_0805_2012Metric, symbol Device:R_Small_US
- added R23: 22, Resistor_SMD:R_0805_2012Metric, symbol Device:R_Small_US
- J2: footprint Connector_PinHeader_2.54mm:PinHeader_1x04_P2.54mm_Horizontal -> Connector_PinHeader_2.54mm:PinHeader_1x04_P2.54mm_Vertical
Connections:
- net +5V: now also R23.1
- net GND: now also Q2.2 (E)
- net jb: now also R22.2
- new net: BZ1.1 (+), D1.1 (K), R23.2
- new net: BZ1.2 (-), D1.2 (A), Q2.3 (C)
- new net: Q2.1 (B), R22.1
- no-connect marks 34 -> 33
